File: hardware/ciphe-decoder-ring.kicad_sch (KiCad schematic)
At the start: 35 parts, among them SW1 EC11E09244BS, U1 XIAO-RP2040-DIP

Commit message: As manufacured with JLCPCB on 2025-Feb-27
Parts:
- added R1: 470, Resistor_SMD:R_0402_1005Metric, symbol Device:R
- added R2, R3: 5.1k, Resistor_SMD:R_0402_1005Metric, symbol Device:R
- added TP1, TP2: TestPoint, TestPoint:TestPoint_Pad_D1.5mm, symbol Connector:TestPoint
Connections:
- net +5V: now also R2.1, R3.2
- net LED_IN: now also R1.2, TP2.1; no longer U1.8 (GPIO1/RX)
- net at SW1.B, U1.1 (GPIO26/ADC0/A0): now also R2.2
- net at SW1.A, U1.2 (GPIO27/ADC1/A1): now also R3.1
- new net: R1.1, TP1.1, U1.8 (GPIO1/RX)

Commit message: Adding schematic as a PDF for review
Other:
- company: (none) -> Steven Smethurst (@Funvill)
- title: (none) -> Cipher Decoder Ring PCB
Changed lines of the file:
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@@
 	(generator_version "9.0")
 	(paper "A4")
+	(title_block
+		(title "Cipher Decoder Ring PCB")
+		(date "2025-02-27")
+		(rev "2024-Feb-27")
+		(company "Steven Smethurst (@Funvill)")
+		(comment 1 "https://github.com/funvill/cipher-decoder-ring-pcb")
+	)
 	(junction
 		(at 90.17 20.32)
